File: AMN_TopPcb/AMN_TopPcb.kicad_pcb (KiCad board)
At the start: 2 copper layers, 93 x 93 mm, 24 parts, among them J5 Debug, J6 UPDI, SW2 SW_DIP_x02, U3 MCP1804x-5002xOT, U4 ATtiny3224-SS

Commit message: 4
Parts:
- removed C5, C6, C7: 100nF, Capacitor_SMD:C_0603_1608Metric
- removed D10: 5v1, Diode_SMD:D_SMF
- removed D11, D9: LED, LED_SMD:LED_0805_2012Metric
- removed J5: Debug, Connector_PinHeader_2.54mm:PinHeader_1x03_P2.54mm_Vertical
- removed J6: UPDI, Connector_PinHeader_2.54mm:PinHeader_1x03_P2.54mm_Vertical
- removed R12, R13: 10k, Resistor_SMD:R_0603_1608Metric
- removed R14, R15: 4k7, Resistor_SMD:R_0603_1608Metric
- removed R16: 2k7, Resistor_SMD:R_0603_1608Metric
- removed R17: 1k5, Resistor_SMD:R_0603_1608Metric
- removed RV3, RV4: 10k, Potentiometer_THT:Potentiometer_Alps_RK09K_Single_Vertical
- removed SW2: SW_DIP_x02, Button_Switch_THT:SW_DIP_SPSTx02_Slide_9.78x7.26mm_W7.62mm_P2.54mm
- removed U3: MCP1804x-5002xOT, Package_TO_SOT_SMD:SOT-23-5
- removed U4: ATtiny3224-SS, Package_SO:SOIC-14_3.9x8.7mm_P1.27mm
- added C1: 100nF, Capacitor_SMD:C_0603_1608Metric, B.Cu at (168.2, 79.5)
- added C2: 100nF, Capacitor_SMD:C_0603_1608Metric, B.Cu at (150.0, 75.4)
- added C3: 10uF, Capacitor_SMD:C_0603_1608Metric, B.Cu at (143.0, 73.5)
- added D1: 5v1, Diode_SMD:D_SMF, B.Cu at (165.8, 81.8)
- added D2: LED, LED_SMD:LED_0805_2012Metric, F.Cu at (126.2, 59.4)
- added D3: LED, LED_SMD:LED_0805_2012Metric, F.Cu at (116.2, 59.4)
- added D4: LED, LED_SMD:LED_0805_2012Metric, F.Cu at (146.2, 59.4)
- added D5: LED, LED_SMD:LED_0805_2012Metric, F.Cu at (136.2, 59.4)
- added D6: LED, LED_SMD:LED_0805_2012Metric, F.Cu at (156.2, 59.4)
- added J1: Debug, Connector_PinHeader_2.54mm:PinHeader_1x03_P2.54mm_Vertical, F.Cu at (158.6, 136.1)
- added J2: UPDI, Connector_PinHeader_2.54mm:PinHeader_1x03_P2.54mm_Vertical, F.Cu at (145.2, 136.0)
- added J3: Conn_02x03_Odd_Even, Connector_PinHeader_2.54mm:PinHeader_2x03_P2.54mm_Vertical, B.Cu at (168.2, 59.4)
- added R1: 4k7, Resistor_SMD:R_0603_1608Metric, B.Cu at (164.9, 79.5)
- added R2: 2k7, Resistor_SMD:R_0603_1608Metric, B.Cu at (164.9, 77.8)
- added R3: 4k7, Resistor_SMD:R_0603_1608Metric, B.Cu at (126.3, 63.9)
- added R4: 10k, Resistor_SMD:R_0603_1608Metric, B.Cu at (128.8, 132.9)
- added R5: 10k, Resistor_SMD:R_0603_1608Metric, B.Cu at (128.9, 138.9)
- added R6: 1k5, Resistor_SMD:R_0603_1608Metric, B.Cu at (116.1, 63.9)
- added R7: 1k5, Resistor_SMD:R_0603_1608Metric, B.Cu at (146.2, 63.9)
- added R8: 1k5, Resistor_SMD:R_0603_1608Metric, B.Cu at (136.1, 63.9)
- added R9: 1k5, Resistor_SMD:R_0603_1608Metric, B.Cu at (156.1, 63.9)
- added RV1: 10k, Potentiometer_THT:Potentiometer_Alps_RK09K_Single_Vertical, F.Cu at (122.5, 106.7)
- added RV2: 10k, Potentiometer_THT:Potentiometer_Alps_RK09K_Single_Vertical, F.Cu at (156.8, 106.8)
- added SW1: SW_DIP_x02, Button_Switch_THT:SW_DIP_SPSTx02_Slide_9.78x7.26mm_W7.62mm_P2.54mm, F.Cu at (116.7, 134.6)
- added U1: ATtiny3224-SS, Package_SO:SOIC-14_3.9x8.7mm_P1.27mm, B.Cu at (139.7, 81.4)
- added U2: MCP1804x-5002xOT, Package_TO_SOT_SMD:SOT-23-5, B.Cu at (148.0, 78.5)
- C4: value 10uF -> 100nF
- moved C4 27.3 mm to (143.0, 75.3), turned to 180 degrees
Routing:
- net +5V: track 0.00 -> 136.0 mm, vias 0 -> 1
- net OFF_Scale: track 0.00 -> 79.9 mm
- net RX: track 0.00 -> 75.9 mm, vias 0 -> 2
- net ON_Scale: track 0.00 -> 75.6 mm
- net TX: track 0.00 -> 75.2 mm, vias 0 -> 2
- net VALVE_OUT: track 0.00 -> 64.6 mm, vias 0 -> 3
- net START_CONN: track 0.00 -> 62.7 mm
- net UPDI: track 0.00 -> 58.7 mm, vias 0 -> 2
- net BLEED_OFF: track 0.00 -> 56.8 mm, vias 0 -> 1
- net RELAY_OUT: track 0.00 -> 53.7 mm, vias 0 -> 3
- net /ON_Time: track 0.00 -> 52.1 mm
- net +12V: track 0.00 -> 45.4 mm, vias 0 -> 1
- net /OFF_Time: track 0.00 -> 41.3 mm, vias 0 -> 1
- net RUN_Led: track 0.00 -> 37.8 mm, vias 0 -> 1
- net START: track 0.00 -> 26.6 mm, vias 0 -> 2
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- added copper zone on B.Cu, net GND
- added copper zone on F.Cu, net GND
Other:
- board text added: "+5V"
- board text added: "0,1 . 1"
- board text added: "1 . 10"
- board text added: "10 . 100"
- board text added: "2 . 20"
- board text added: "20 . 200"
- board text added: "3 . 30"
- board text added: "30 . 300"
- board text added: "GND"
- board text added: "MIN"
- board text added: "OFF"
- board text added: "OFF TID"
- board text added: "OFF TID i Minutter"
- board text added: "ON"
- board text added: "ON TID"
- board text added: "ON TID i Sekunder"
- board text added: "RELAY"
- board text added: "RL 1"
- board text added: "RL 2"
- board text added: "RUN"
- board text added: "RX"
- board text added: "SEK"
- board text added: "START"
- board text added: "TX"
- board text added: "UPDI"
