File: AMN_TopPcb/AMN_TopPcb.kicad_sch (KiCad schematic)
At the start: 21 parts, among them J5 Debug, J6 UPDI, J7 Screw_Terminal_01x04, SW2 SW_DIP_x02, U3 MCP1804x-5002xOT, U4 ATtiny3224-SS

Commit message: 1
Parts:
- removed J7: Screw_Terminal_01x04, Connector_Phoenix_MC:PhoenixContact_MCV_1,5_4-G-3.5_1x04_P3.50mm_Vertical, symbol Connector:Screw_Terminal_01x04
- added H1, H2, H3, H4: MountingHole, MountingHole:MountingHole_3.5mm, symbol Mechanical:MountingHole
- D11: footprint (none) -> LED_SMD:LED_0805_2012Metric
- D9: footprint LED_SMD:LED_1206_3216Metric -> LED_SMD:LED_0805_2012Metric
- R17: footprint (none) -> Resistor_SMD:R_0603_1608Metric
- RV3, RV4: footprint (none) -> Potentiometer_THT:Potentiometer_Alps_RK09K_Single_Vertical
- SW2: footprint (none) -> Button_Switch_THT:SW_DIP_SPSTx02_Slide_9.78x7.26mm_W7.62mm_P2.54mm
Connections:
- net GND: now also C4.1, C5.1, U3.2 (GND)

Commit message: 3
Connections:
- net at U3.1 (VIN): now also U3.4 (~{SHDN})
Changed lines of the file:
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@@
+	(wire
+		(pts
+			(xy 293.37 92.71) (xy 290.83 92.71)
+		)
+		(stroke
+			(width 0)
+			(type default)
+		)
+	)
 	(wire
 		(pts
@@
 	(wire
 		(pts
+			(xy 290.83 90.17) (xy 293.37 90.17)
+		)
+		(stroke
+			(width 0)
+			(type default)
+		)
+	)
+	(wire
+		(pts
 			(xy 158.75 91.44) (xy 158.75 92.71)
 		)
@@
 		)
 		(stroke
+			(width 0)
+			(type default)
+		)
+	)
+	(wire
+		(pts
+			(xy 290.83 92.71) (xy 290.83 90.17)
+		)
+		(stroke

Commit message: 4
Parts:
- added D4, D5, D6: LED, LED_SMD:LED_0805_2012Metric, symbol Device:LED
- added J3: Conn_02x03_Odd_Even, Connector_PinHeader_2.54mm:PinHeader_2x03_P2.54mm_Vertical, symbol Connector_Generic:Conn_02x03_Odd_Even
- added R7, R8, R9: 1k5, Resistor_SMD:R_0603_1608Metric, symbol Device:R_Small
- RV1: renamed from RV3; symbol Device:R_Potentiometer -> Device:R_Potentiometer_MountingPin
- RV2: renamed from RV4; symbol Device:R_Potentiometer -> Device:R_Potentiometer_MountingPin
- renumbered C7 to C1, C6 to C2, C4 to C3, C5 to C4, D10 to D1, D9 to D2, D11 to D3, J5 to J1, J6 to J2, R15 to R1, R16 to R2, R14 to R3, R13 to R4, R12 to R5, R17 to R6, SW2 to SW1, U4 to U1, U3 to U2
Connections:
- net +12V: now also U2.1 (VIN), U2.4 (~{SHDN}), J3.1 (Pin_1)
- net GND: now also RV1.MP (MountPin), RV2.MP (MountPin), J3.3 (Pin_3), R7.2, R8.2, R9.2
- net OFF_Scale: now also U1.9 (PB0); no longer U1.8 (PB1)
- net ON_Scale: now also U1.8 (PB1); no longer U1.9 (PB0)
- net RX: now also J1.3 (Pin_3); no longer J1.2 (Pin_2)
- net TX: now also J1.2 (Pin_2); no longer J1.3 (Pin_3)
- net START_CONN: now reaches C1.1, R1.2, R3.2
- net START_CONN: now also J3.5 (Pin_5)
- net BLEED_OFF: now reaches U1.11 (PA1)
- net BLEED_OFF: now also D5.2 (A), J3.4 (Pin_4)
- net VALVE_OUT: now reaches U1.12 (PA2)
- net VALVE_OUT: now also D4.2 (A), J3.2 (Pin_2)
- net RELAY_OUT: now reaches U1.13 (PA3)
- net RELAY_OUT: now also D6.2 (A), J3.6 (Pin_6)
- new net: D5.1 (K), R8.1
- new net: D4.1 (K), R7.1
- new net: D6.1 (K), R9.1
